Commit message: feat: add Debug Mode setting, remove noisy logs
Debug Mode:
- Added ui.debug_mode checkbox in Settings page
- Performance menu and Debug menu only visible when enabled
- Record Performance toggle only visible when enabled
- Console debug logs only output when enabled
- IK Axis Mask selector only shown when enabled

Other:
- Removed noisy "Broadcasting system metrics" log from API

🤖 Generated with [Claude Code](https://claude.com/claude-code)

Co-Authored-By: Claude <noreply@anthropic.com>

File: frontend/public/urdf/PAROL6.urdf (robot description, URDF)
Before this commit: robot parol6, 8 links, 7 joints
Joints:
- joint L4: origin xyz=-0.0435 0.17635 0 rpy=1.5707963267949 0 0 -> xyz=-0.0435 0.17635 0 rpy=1.5707963267949 -1.5707963267949 0
